Commit message: Added demo video

File: src/dof4_arm_description/urdf/dof4_arm.urdf (robot description, URDF)
Before this commit: robot dof4_arm, 5 links, 4 joints
Links:
- added link gripper_base; visual box size=0.1 0.06 0.06
- added link left_finger; visual box size=0.08 0.02 0.02
- added link object_box; visual box size=0.06 0.06 0.06
- added link place_box; visual box size=0.1 0.1 0.04
- added link right_finger; visual box size=0.08 0.02 0.02
- link base_link: geometry visual box size=0.4 0.4 0.1
- link link1: geometry visual cylinder length=0.4 radius=0.05
- link link2: geometry visual box size=0.6 0.1 0.1
- link link3: geometry visual box size=0.5 0.08 0.08
- link link4: geometry visual box size=0.4 0.07 0.07
Joints:
- added joint gripper_base_joint: type fixed, parent link4, child gripper_base, origin xyz=0.3 0 0
- added joint left_finger_joint: type prismatic, parent gripper_base, child left_finger, origin xyz=0 0.02 0, axis 0 1 0, limit lower=0.0 upper=0.04 effort=10 velocity=0.2
- added joint object_fixed: type fixed, parent gripper_base, child object_box, origin xyz=0.05 0 0
- added joint place_fixed: type fixed, parent gripper_base, child place_box, origin xyz=0.05 0 0
- added joint right_finger_joint: type prismatic, parent gripper_base, child right_finger, origin xyz=0 -0.02 0, axis 0 -1 0, limit lower=0.0 upper=0.04 effort=10 velocity=0.2
- joint joint2: limit lower=-3.14 upper=3.14 effort=10 velocity=1 -> lower=-1.57 upper=1.57 effort=10 velocity=1; origin xyz=0 0 0.1 -> xyz=0 0 0.4
- joint joint3: limit lower=-3.14 upper=3.14 effort=10 velocity=1 -> lower=-1.57 upper=1.57 effort=10 velocity=1; origin xyz=0 0 0.1 -> xyz=0.6 0 0
- joint joint4: axis 0 1 0 -> 1 0 0; origin xyz=0 0 0.1 -> xyz=0.5 0 0
